File: rp2040-pcb.kicad_pcb (KiCad board)
At the start: 2 copper layers, 0 parts

Commit message: Started routing.
Parts:
- added C1: 10µ, Capacitor_SMD:C_0603_1608Metric, F.Cu at (384.2, -86.7)
- added C10: 1µ, Capacitor_SMD:C_0603_1608Metric, F.Cu at (370.8, -84.4)
- added C11: 100n, Capacitor_SMD:C_0402_1005Metric, F.Cu at (372.6, -76.6)
- added C12: 100n, Capacitor_SMD:C_0402_1005Metric, F.Cu at (377.7, -80.5)
- added C13: 100n, Capacitor_SMD:C_0402_1005Metric, F.Cu at (377.7, -78.5)
- added C14: 100n, Capacitor_SMD:C_0402_1005Metric, F.Cu at (372.0, -80.5)
- added C15: 100n, Capacitor_SMD:C_0402_1005Metric, F.Cu at (374.9, -78.5)
- added C16: 100n, Capacitor_SMD:C_0402_1005Metric, F.Cu at (380.6, -80.5)
- added C17: 100n, Capacitor_SMD:C_0402_1005Metric, F.Cu at (372.0, -78.5)
- added C18: 100n, Capacitor_SMD:C_0402_1005Metric, F.Cu at (374.9, -80.5)
- added C19: 27p, Capacitor_SMD:C_0402_1005Metric, F.Cu at (369.1, -80.0)
- added C2: 100n, Capacitor_SMD:C_0402_1005Metric, F.Cu at (369.1, -82.0)
- added C20: 27p, Capacitor_SMD:C_0402_1005Metric, F.Cu at (366.8, -76.1)
- added C3: 100n, Capacitor_SMD:C_0402_1005Metric, F.Cu at (363.9, -78.0)
- added C4: 22µ, Capacitor_SMD:C_0805_2012Metric, F.Cu at (375.5, -89.0)
- added C5: 22µ, Capacitor_SMD:C_0805_2012Metric, F.Cu at (371.1, -89.0)
- added C6: 56p, Capacitor_SMD:C_0402_1005Metric, F.Cu at (366.8, -78.0)
- added C7: 100n, Capacitor_SMD:C_0402_1005Metric, F.Cu at (369.7, -76.6)
- added C8: 100n, Capacitor_SMD:C_0402_1005Metric, F.Cu at (361.1, -76.6)
- added C9: 1µ, Capacitor_SMD:C_0603_1608Metric, F.Cu at (366.8, -84.2)
- added J1: Conn_01x20_Male, Connector_PinHeader_2.54mm:PinHeader_1x20_P2.54mm_Vertical, F.Cu at (338.5, -88.2)
- added J2: Conn_01x20_Male, Connector_PinHeader_2.54mm:PinHeader_1x20_P2.54mm_Vertical, F.Cu at (403.0, -85.1)
- added J3: USB_C_Receptacle, Connector_USB:USB_C_Receptacle_Palconn_UTC16-G, F.Cu at (370.0, -36.0)
- added L1: 10µ, Inductor_SMD:L_0603_1608Metric, F.Cu at (384.2, -89.2)
- added PWR_LED1: RED, LED_SMD:LED_0805_2012Metric, F.Cu at (380.0, -89.0)
- added R1: 56, Resistor_SMD:R_0402_1005Metric, F.Cu at (374.3, -86.5)
- added R10: 5.1k, Resistor_SMD:R_0402_1005Metric, F.Cu at (377.2, -84.5)
- added R11: 5.1k, Resistor_SMD:R_0402_1005Metric, F.Cu at (380.1, -84.5)
- added R12: 1k, Resistor_SMD:R_0402_1005Metric, F.Cu at (380.1, -82.5)
- added R2: 100k, Resistor_SMD:R_0402_1005Metric, F.Cu at (377.2, -86.5)
- added R3: 22k, Resistor_SMD:R_0402_1005Metric, F.Cu at (383.0, -84.5)
- added R4: 680, Resistor_SMD:R_0402_1005Metric, F.Cu at (383.0, -82.5)
- added R5: 27.4, Resistor_SMD:R_0402_1005Metric, F.Cu at (366.2, -80.5)
- added R6: 27.4, Resistor_SMD:R_0402_1005Metric, F.Cu at (380.1, -86.5)
- added R7: 10k, Resistor_SMD:R_0402_1005Metric, F.Cu at (374.3, -84.5)
- added R8: 1k, Resistor_SMD:R_0402_1005Metric, F.Cu at (374.3, -82.5)
- added R9: 10k, Resistor_SMD:R_0402_1005Metric, F.Cu at (377.2, -82.5)
- added SW1: SW_Push, Button_Switch_SMD:SW_SPST_TL3342, F.Cu at (381.0, -41.0)
- added SW2: SW_Push, Button_Switch_SMD:SW_SPST_TL3342, F.Cu at (351.0, -37.0)
- added U1: TPS54202DDC, Package_TO_SOT_SMD:SOT-23-6, F.Cu at (362.2, -81.2)
- added U2: W25Q128JVSIQ, Package_SO:SOIC-8_5.23x5.23mm_P1.27mm, F.Cu at (389.0, -73.0)
- added U3: RP2040, Package_DFN_QFN:QFN-56-1EP_7x7mm_P0.4mm_EP3.2x3.2mm_ThermalVias, F.Cu at (369.0, -58.0)
- added Y1: 12 MHz, Oscillator:Oscillator_SMD_EuroQuartz_XO32-4Pin_3.2x2.5mm, F.Cu at (366.8, -88.1)
